File: F405Pill_V2/F405Pill_V2.sch (KiCad schematic (older format))
At the start: 35 parts, among them J1 USB_A, J2 Conn_01x04, J3 Conn_01x20, J4 Conn_01x20, SW1 SW_Push, U1 STM32F411RETx, U2 MCP1703A-3302_SOT223, Y1 8MHz, Y2 32kHz

Commit message: Abandoned this project as uneconomic, but commited file all my incomplete work in case its of value to anyone else
Parts:
- removed U1: STM32F411RETx, Housings_QFP:LQFP-64_7x7mm_Pitch0.4mm, symbol STM32F411RETx
- added C15: 10u, Capacitors_SMD:C_0603, symbol C
- added U1: STM32F405RGTx, BluePill_Specials:LQFP-64-1EP_10x10mm_Pitch0.5mm_SPECIAL, symbol STM32F405RGTx
- added U3: MCP1703A-3302_SOT223, TO_SOT_Packages_SMD:SC-70, symbol MCP1703A-3302_SOT223
- L1: footprint Inductors:Inductor_Taiyo-Yuden_MD-1616 -> Inductors:Inductor_Taiyo-Yuden_MD-5050
- SW1: footprint Buttons_Switches_SMD:SW_DIP_x1_W5.08mm_Slide_Copal_CHS-A -> Buttons_Switches_SMD:SW_SPST_B3S-1000
- U2: footprint TO_SOT_Packages_SMD:SOT-223-3Lead_TabPin2 -> TO_SOT_Packages_SMD:SC-70
- Y1, Y2: footprint Crystals:Crystal_HC52-6mm_Vertical -> Crystals:Crystal_HC18-U_Vertical
Connections:
- net labels added: VCCA3V3
- net labels removed: SWCLK, SWDIO
- wire segments 171 -> 179
Other:
- moved on the sheet: R8
