File: Squonk42/BluePillF4.sch (KiCad schematic (older format))
At the start: 54 parts, among them J1 MH20-1, J2 MH20-1, J3 MH_RA4-1, J4 MR07C-06200, J5 47642-001, Q1 DMP2160UW-7, U1 AP2114HA-3.3TRG1, U2 AP2112K3.3-TRG1, U3 STM32F405RGT6, U4 SY6280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

Commit message: Remove FET between VBus and +5V and replace with Schottky diode
Parts:
- removed Q1: DMP2160UW-7, BluePillF4 0603 TD:SOT323, symbol DMP2160UW-7
- added D3: SS12, Diodes_SMD:D_SMA, symbol SS12
Connections:
- wire segments 257 -> 256

Commit message: Revert back to commit 7277910...
Parts:
- removed D3: SS12, Diodes_SMD:D_SMA, symbol SS12
- added Q1: DMP2160UW-7, BluePillF4 0603 TD:SOT323, symbol DMP2160UW-7
Connections:
- wire segments 256 -> 257

Commit message: Powered AP2112 from +5V, not from +3.3V Added ferrite bead between GND and AGND Replaced 32kHz crystal by smaller FC-12M Adjusted solder mask clearance to 0 Made VBAT trace thinner Fixed MOSFET direction => replaced by an 1N5819HW Schottky diode Added PWR_FLAG to schematic to remove ERC warnings Replaced NC by real Kicad ones to remove ERC warnings Cleaned up Expansion connector labels in schematic Cleaned up traces for PA13-14 and PC13-15 Changed micro USB connector to BSC-Elec U02-BFD3111B0-009
Parts:
- removed Q1: DMP2160UW-7, BluePillF4 0603 TD:SOT323, symbol DMP2160UW-7
- removed Y1: FC-135, BluePillF4 0603 TD:CRYSTAL_32X15, symbol FC-135
- added D3: 1N5819HW, BluePillF4 Lib:SOD-123, symbol 1N5819HW
- added L2: BLM18BA470SN1D, BluePillF4 Lib:FB0603, symbol FB_0603
- added Y1: FC-12M, BluePillF4 Lib:FC-12M, symbol FC-12M
- C1, C10, C11, C12, C13, C14, C15, C16, C17, C2, C3, C4, C5, C6, C7, C8, C9: footprint BluePillF4 0603 TD:C0603 -> BluePillF4 Lib:C0603
- D1, D2: footprint BluePillF4 0603 TD:LED0603 -> BluePillF4 Lib:LED0603
- J1, J2: footprint BluePillF4 0603 TD:MH20-1-0.1 -> BluePillF4 Lib:MH20-1-0.1
- J3: footprint BluePillF4 0603 TD:MH_RA4-1-0.1 -> BluePillF4 Lib:MH_RA4-1-0.1
- J4: footprint BluePillF4 0603 TD:MR07C-06200 -> BluePillF4 Lib:MR07C-06200
- J5: value 47642-001 -> U02-BFD3111B0-009; footprint BluePillF4 0603 TD:47662-001 -> BluePillF4 Lib:U02-BFD3111B0-009; symbol 47642-001 -> U02-BFD3111B0-009
- L1: footprint BluePillF4 0603 TD:FB0603 -> BluePillF4 Lib:FB0603
- PC0, PC1, PC2, PC3, PC5, PC6, PC7: footprint BluePillF4 0603 TD:TEST_PAD -> BluePillF4 Lib:TEST_PAD
- R1, R10, R11, R12, R13, R2, R3, R4, R5, R6, R7, R8, R9: footprint BluePillF4 0603 TD:R0603 -> BluePillF4 Lib:R0603
- S1, S2: footprint BluePillF4 0603 TD:SKSGACE010 -> BluePillF4 Lib:SKSGACE010
- U1: footprint BluePillF4 0603 TD:SOT223 -> BluePillF4 Lib:SOT223
- U2, U4: footprint BluePillF4 0603 TD:SOT23-5 -> BluePillF4 Lib:SOT23-5
- U3: footprint BluePillF4 0603 TD:LQFP64 -> BluePillF4 Lib:LQFP64
- Y2: footprint BluePillF4 0603 TD:CRYSTAL_32X25_2P -> BluePillF4 Lib:CRYSTAL_32X25_2P
Connections:
- net labels removed: ~
- wire segments 257 -> 261
- no-connect marks 0 -> 4
Other:
- moved on the sheet: C1, C10, C11, C12, C13, C14, C15, C16, C17, C2, C3, C4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
