File: Squonk42/BluePillF4-1.sch (KiCad schematic (older format))
At the start: 61 parts, among them J1 MH20-1, J2 MH20-1, J3 MH_RA4-1, J4 MR07C-06200, J5 U02-BFD3111B0-009, U1 AP2114HA-3.3TRG1, U2 AP2112K3.3-TRG1, U3 STM32F405RGT6, U4 SY6280, Y1 FC-12M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

Commit message: Replaced the MicroSD Card connector with a Molex 47309-2651 Added voltage sense resistor divider Cleaned up traces
Parts:
- removed C18: 100n, BluePillF4 Lib:C0603, symbol CAP_0603
- removed C6, C8: 4u7, BluePillF4 Lib:C0603, symbol CAP_0603
- removed U1: AP2114HA-3.3TRG1, BluePillF4 Lib:SOT223, symbol AP2114HA-3.3TRG1
- removed U2: AP2112K3.3-TRG1, BluePillF4 Lib:SOT23-5, symbol AP2112K3.3-TRG1
- added R21, R22: 10k, BluePillF4 Lib:R0603, symbol RES_0603
- C1, C10, C11, C12, C13, C14, C15, C16, C17, C2, C3, C4, C5, C7, C9: AliExpress (none) -> https://www.aliexpress.com/item/0603-SMD-Capacitor-assorted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
- D1: AliExpress (none) -> https://www.aliexpress.com/item/100pcs-lot-5-Colors-0603-SM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
- D2: AliExpress (none) -> https://www.aliexpress.com/item/100-pcs-0603-1616-RGB-LED-A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
- D3: AliExpress (none) -> https://www.aliexpress.com/item/Livraison-gratuite-100-pcs-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
- J1, J2, J3, PC1, PC2, PC3, PC4, PC5, PC6, PC7: AliExpress (none) -> N/A
- J4: value MR07C-06200 -> 47309-2651; footprint BluePillF4 Lib:MR07C-06200 -> BluePillF4 Lib:47309-2651; symbol MR07C-06200 -> 47309-2651; AliExpress (none) -> https://fr.aliexpress.com/item/10-PCS-LOT-Court-TF-carte-mi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; HEIGHT 1.9mm -> 2.65mm; PARTNO MR07C-06200 -> 47309-2651
- J5: AliExpress (none) -> https://www.aliexpress.com/item/50pcs-Micro-USB-Connector-5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
- L2: AliExpress (none) -> https://www.aliexpress.com/item/100PCS-0603-47R-47-ohm-SMD-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
- R1, R10, R11, R13, R16, R4, R6, R7, R9: AliExpress (none) -> https://www.aliexpress.com/item/Free-shipping-0603-SMD-Resi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
- R12, R14, R2, R20, R3, R5, R8: AliExpress (none) -> https://www.aliexpress.com/item/300-pcs-lot-SMD-Puce-R-sist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
- R15: AliExpress (none) -> https://www.aliexpress.com/store/product/300-pcs-lot-SMD-Pu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
- S1, S2: AliExpress (none) -> https://www.aliexpress.com/item/3-5-2-7-1-4-Micro-Switch-bu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
- U3: AliExpress (none) -> https://www.aliexpress.com/item/QFP-STM32F405-STM32F405RGT6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
- U4: AliExpress (none) -> https://www.aliexpress.com/item/20PCS-SY6280AAC-SY6280AA-SY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
- Y1: AliExpress (none) -> https://www.aliexpress.com/item/Free-shipping-10pcs-Passive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
- Y2: AliExpress (none) -> https://www.aliexpress.com/item/Passive-small-size-3225-2-f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
Connections:
- wire segments 273 -> 261
- no-connect marks 4 -> 6
Other:
- note added: "Note: PC14/PC15 shared\nbetween LSE clock and\nExpansion"
- note added: "VOLTAGE\nSENSE"
- note removed: "Note: PC14/PC15 shared\nbetween HSE clock and\nExpansion"
- note removed: "POWER"
- moved on the sheet: D1, D2, R14, R15, R2, R3
