File: Squonk42/KiCAD/BluePillF4-1.sch (KiCad schematic (older format))
At the start: 58 parts, among them J1 MH20-1, J2 MH20-1, J3 MH_RA4-1, J4 47309-2651, J5 U02-BFD3111B0-009, U3 STM32F405RGT6, U4 SY6280, Y1 FC-12M, Y2 NX3225GD

Commit message: added EagleCAD version
Parts:
- removed R6: 10k, BluePillF4 Lib:R0603, symbol RES_0603
- C1, C10, C11, C12, C13, C14, C15, C16, C17, C2, C3, C4, C5, C7, C9: symbol CAP_0603 -> BluePillF4:CAP_0603
- D1: symbol LED_0603 -> BluePillF4:LED_0603
- D2: symbol 1616RGB -> BluePillF4:1616RGB
- D3: symbol 1N5819HW -> BluePillF4:1N5819HW
- J1, J2: symbol MH20-1 -> BluePillF4:MH20-1
- J3: symbol MH_RA4-1 -> BluePillF4:MH_RA4-1
- J4: symbol 47309-2651 -> BluePillF4:47309-2651
- J5: symbol U02-BFD3111B0-009 -> BluePillF4:U02-BFD3111B0-009
- L1, L2: symbol FB_0603 -> BluePillF4:FB_0603
- L3: symbol FB_0805 -> BluePillF4:FB_0805
- PC1, PC2, PC3, PC4, PC5, PC6, PC7: symbol TEST_PAD -> BluePillF4:TEST_PAD
- R1, R10, R11, R12, R13, R14, R15, R16, R2, R20, R3, R4, R5, R7, R8, R9: symbol RES_0603 -> BluePillF4:RES_0603
- R21, R22: symbol RES_0603 -> BluePillF4:RES_0603; PARTNO R0603_10k_5%_125mW -> R0603_10k_1%_125mW; TOL 5% -> 1%
- S1, S2: symbol SKSGACE010 -> BluePillF4:SKSGACE010
- U3: symbol STM32F405RGT6 -> BluePillF4:STM32F405RGT6
- U4: symbol SY6280 -> BluePillF4:SY6280
- Y1: symbol FC-12M -> BluePillF4:FC-12M
- Y2: symbol NX3225GD -> BluePillF4:NX3225GD
Connections:
- net labels removed: R6
- wire segments 261 -> 311
