File: Squonk42/KiCAD/BluePillF4-2.sch (KiCad schematic (older format))
At the start: 13 parts, among them Q1 IRLML6402, U1 AP2114HA-3.3TRG1, U2 AP2112K3.3-TRG1, U5 MCP73812T-420I/OT

Commit message: added EagleCAD version
Parts:
- C18, C19, C20, C6, C8: symbol CAP_0603 -> BluePillF4:CAP_0603
- D4: symbol 1N5819HW -> BluePillF4:1N5819HW
- Q1: symbol IRLML6402 -> BluePillF4:IRLML6402
- R17, R18, R19: symbol RES_0603 -> BluePillF4:RES_0603
- U1: symbol AP2114HA-3.3TRG1 -> BluePillF4:AP2114HA-3.3TRG1
- U2: symbol AP2112K3.3-TRG1 -> BluePillF4:AP2112K3.3-TRG1
- U5: symbol MCP73812T-420I/OT -> BluePillF4-rescue:MCP73812T-420I_OT
Connections:
- wire segments 38 -> 60
Changed lines of the file:
@@
-EESchema Schematic File Version 2
-LIBS:BluePillF4
-LIBS:power
+EESchema Schematic File Version 4
 LIBS:BluePillF4-cache
-EELAYER 25 0
+EELAYER 26 0
 EELAYER END
 $Descr A4 11693 8268
@@
 $Bitmap
 Pos 8100 6800
-Scale 1,000000
+Scale 1.000000
 Data
 89 50 4E 47 0D 0A 1A 0A 00 00 00 0D 49 48 44 52 00 00 01 93 00 00 00 8D 08 06 00 00 00 72 B7 97
@@
 $EndBitmap
 $Comp
-L RES_0603 R?
+L BluePillF4:RES_0603 R?
 U 1 1 5A4D9DD1
 P 1700 1200
@@
 $EndComp
 $Comp
-L 1N5819HW D?
+L BluePillF4:1N5819HW D?
 U 1 1 5A4DA4E6
 P 3200 1300
@@
 $EndComp
 $Comp
-L RES_0603 R?
+L BluePillF4:RES_0603 R?
 U 1 1 5A4DB01E
 P 3000 2500
@@
 $EndComp
 $Comp
-L RES_0603 R?
+L BluePillF4:RES_0603 R?
 U 1 1 5A4DB032
 P 2300 2500
@@
 $EndComp
 $Comp
-L CAP_0603 C?
+L BluePillF4:CAP_0603 C?
 U 1 1 5A4DC5F8
 P 1100 2500
@@
 $EndComp
 $Comp
-L CAP_0603 C?
+L BluePillF4:CAP_0603 C?
 U 1 1 5A4DC654
 P 2600 2500
@@
 $EndComp
 $Comp
-L MCP73812T-420I/OT U5
+L BluePillF4-rescue:MCP73812T-420I_OT U5
 U 1 1 5A4DC6E1
 P 1700 2100
+AR Path="/5A4DC6E1" Ref="U5"  Part="1"
+AR Path="/5A4D7C11/5A4DC6E1" Ref="U5"  Part="1"
 F 0 "U5" H 1300 2500 70  0000 L BNN
 F 1 "MCP73812T-420I/OT" H 1500 2500 70  0000 L BNN
@@
 $EndComp
 $Comp
-L +VIN #SUPPLY047
+L BluePillF4:+VIN #SUPPLY047
 U 1 1 5A4DC75E
 P 3400 1100
@@
 $EndComp
 $Comp
-L +5V #SUPPLY048
+L BluePillF4:+5V #SUPPLY048
 U 1 1 5A4DC787
 P 1100 1100
@@
 $EndComp
 $Comp
-L GND #SUPPLY049
+L BluePillF4:GND #SUPPLY049
 U 1 1 5A4DC7A9
 P 1700 2900
@@
 $EndComp
 $Comp
-L IRLML6402 Q1
+L BluePillF4:IRLML6402 Q1
 U 1 1 5A4DC942
 P 3400 1600
@@
 Ceramic capacitors are +-10% 50V X7R dielectric 0603 unless otherwise specified
 $Comp
-L +VBAT #SUPPLY050
+L BluePillF4:+VBAT #SUPPLY050
 U 1 1 5A587EA2
 P 4300 1800
@@
 Note: Mount L1\nor U2, but not\nboth
 $Comp
-L CAP_0603 C?
+L BluePillF4:CAP_0603 C?
 U 1 1 5A6DFFB9
 P 5450 1450
@@
 $EndComp
 $Comp
-L CAP_0603 C?
+L BluePillF4:CAP_0603 C?
 U 1 1 5A6DFFC7
 P 6450 1450
@@
 $EndComp
 $Comp
-L GND #SUPPLY?
+L BluePillF4:GND #SUPPLY?
 U 1 1 5A6DFFCE
 P 5950 1950
@@
 $EndComp
 $Comp
-L +3V3 #SUPPLY?
+L BluePillF4:+3V3 #SUPPLY?
 U 1 1 5A6DFFD4
 P 6450 1150
@@
 $EndComp
 $Comp
-L +3V3A #SUPPLY?
+L BluePillF4:+3V3A #SUPPLY?
 U 1 1 5A6DFFDA
 P 8250 1150
@@
 $EndComp
 $Comp
-L AP2114HA-3.3TRG1 U?
+L BluePillF4:AP2114HA-3.3TRG1 U?
 U 1 1 5A6DFFE5
 P 5950 1450
@@
 $EndComp
 $Comp
-L AP2112K3.3-TRG1 U?
+L BluePillF4:AP2112K3.3-TRG1 U?
 U 1 1 5A6DFFF1
 P 7750 1450
@@
 $EndComp
 $Comp
-L CAP_0603 C?
+L BluePillF4:CAP_0603 C?
 U 1 1 5A6E0015
 P 6750 1450
@@
 $EndComp
 $Comp
-L +VIN #SUPPLY?
+L BluePillF4:+VIN #SUPPLY?
 U 1 1 5A6E001F
 P 5450 1150
@@
 $EndComp
 $Comp
-L +VIN #SUPPLY?
+L BluePillF4:+VIN #SUPPLY?
 U 1 1 5A6E0025
 P 7250 1150
@@
 $EndComp
 $Comp
-L PWR_FLAG #FLG056
+L power:PWR_FLAG #FLG056
 U 1 1 5A6E002B
 P 5350 1250
@@
 +VIN
 $Comp
-L AGND #SUPPLY?
+L BluePillF4:AGND #SUPPLY?
 U 1 1 5A6E0034
 P 7750 1950
@@
 	2300 2200 2300 2300
 Wire Wire Line
-	2200 1900 4300 1900
-Wire Wire Line
-	1100 2800 3000 2800
+	2200 1900 2600 1900
+Wire Wire Line
+	1100 2800 1700 2800
 Wire Wire Line
 	2300 2700 2300 2800
 Connection ~ 2300 2800
 Wire Wire Line
-	1700 2400 1700 2900
+	1700 2400 1700 2800
 Connection ~ 1700 2800
 Wire Wire Line
 	1100 2800 1100 2600
 Wire Wire Line
-	1100 1100 1100 2400
+	1100 1100 1100 1200
 Wire Wire Line
 	1100 2200 1200 2200
@@
 Connection ~ 1100 2200
 Wire Wire Line
-	1100 1500 3200 1500
-Wire Wire Line
-	3000 1300 3000 2300
+	1100 1500 3000 1500
+Wire Wire Line
+	3000 1300 3000 1500
 Connection ~ 1100 1900
 Wire Wire Line
@@
 	3400 1300 3300 1300
 Wire Wire Line
-	3400 1100 3400 1400
+	3400 1100 3400 1200
 Connection ~ 3400 1300
 Connection ~ 3400 1200
@@
 	2250 600  1450 600
 Wire Wire Line
-	6450 1150 6450 1350
+	6450 1150 6450 1250
 Connection ~ 6450 1250
 Wire Wire Line
@@
 	8250 1250 8250 1150
 Wire Wire Line
-	5350 1250 5550 1250
-Wire Wire Line
-	5450 1150 5450 1350
+	5350 1250 5450 1250
+Wire Wire Line
+	5450 1150 5450 1250
 Connection ~ 5450 1250
 Wire Wire Line
 	5450 1550 5450 1850
 Wire Wire Line
-	5450 1850 6750 1850
-Wire Wire Line
-	5950 1750 5950 1950
+	5450 1850 5950 1850
+Wire Wire Line
+	5950 1750 5950 1850
 Wire Wire Line
 	6450 1850 6450 1550
@@
 Wire Notes Line
 	8650 2250 7150 2250
-Wire Notes Line
-	7150 2250 7150 750
 Wire Wire Line
 	7250 1250 7350 1250
 Connection ~ 7250 1250
 Wire Wire Line
-	6350 1250 6750 1250
-Wire Notes Line
-	7150 765  7150 655
+	6350 1250 6450 1250
 Wire Notes Line
 	7150 655  8650 655
@@
 Connection ~ 6450 1850
 Wire Wire Line
-	7250 1145 7250 1550
+	7250 1145 7250 1250
 Wire Wire Line
 	7250 1550 7350 1550
 Wire Notes Line
 	8700 3250 8700 475
+Wire Wire Line
+	2300 2800 2600 2800
+Wire Wire Line
+	1700 2800 2300 2800
+Wire Wire Line
+	1700 2800 1700 2900
+Wire Wire Line
+	2600 2800 3000 2800
+Wire Wire Line
+	1100 2200 1100 2400
+Wire Wire Line
+	1100 1900 1100 2200
+Wire Wire Line
+	1100 1500 1100 1900
+Wire Wire Line
+	1100 1200 1100 1500
+Wire Wire Line
+	3000 1500 3200 1500
+Wire Wire Line
+	3000 1500 3000 2300
+Wire Wire Line
+	2600 1900 3400 1900
+Wire Wire Line
+	3400 1900 4300 1900
+Wire Wire Line
+	3400 1300 3400 1400
+Wire Wire Line
+	3400 1200 3400 1300
+Wire Wire Line
+	6450 1250 6450 1350
+Wire Wire Line
+	6450 1250 6750 1250
+Wire Wire Line
+	5450 1250 5550 1250
+Wire Wire Line
+	5450 1250 5450 1350
+Wire Wire Line
+	5950 1850 6450 1850
+Wire Wire Line
+	5950 1850 5950 1950
+Wire Wire Line
+	7250 1250 7250 1550
+Wire Wire Line
+	6450 1850 6750 1850
+Wire Notes Line
+	7150 655  7150 2250
 $EndSCHEMATC
